File: electrical-schema/kicad.kicad_sch (KiCad schematic)
At the start: 7 parts, among them U1 ESP32-CAM, U2 AS5600

Commit message: docs: finish electrical schema
Parts:
- added A2, A3: NodeMCU, 113990105:SEEED_113990105, symbol ESP8266:113990105
- added ACC2, ACC3: GY-521, symbol GY-521:GY-521
- added AE1: Antenna, symbol Device:Antenna
- added BuckConverter1, BuckConverter2, BuckConverter3: ~, symbol MIT_Lib:Buck_Converter
- added FTDI_USB_Serial1: ~, symbol MIT_Lib:FTDI_USB_Serial
- added IBT1, IBT4: ~, symbol MIT_Lib:IBT4
- added M1, M3: DNS15, symbol Motor:Motor_Servo
- added M2, M4: Motraxx SR545SA, symbol Motor:Motor_DC
- added PositionSensor, PositionSensor1: AS5600, AS5600:AS5600, symbol AS5600:AS5600
- added STM32_FOC2, STM32_FOC3: ~, symbol MIT_Lib:STM32_FOC
- added TOF400F1, TOF400F2, TOF400F3: ~, symbol MIT_Lib:TOF400F
- added U3: ESP32-CAM, ESP32-CAM:ESP32-CAM, symbol ESP32-CAM:ESP32-CAM
Connections:
- net at U1.P$1 (5V): now also A3.J1_15 (VIN), BuckConverter3. (VOUT-), M3.3 (+)
- net at U1.P$12 (3V3.): now also TOF400F1. (VIN), TOF400F2. (VIN), TOF400F3. (VIN)
- net at U1.P$2 (GND): now also A3.J1_10 (GND), A3.J1_14 (GND), BuckConverter3. (VOUT-), IBT1. (VIN-), M3.4 (-)
- net at U1.P$5 (IO15): now also TOF400F1. (VIN), TOF400F2. (VIN), TOF400F3. (VIN)
- net at U1.P$6 (IO14): now also TOF400F1. (VIN), TOF400F2. (VIN), TOF400F3. (VIN)
- net at U1.P$9 (.GND): now also TOF400F1. (VIN), TOF400F2. (VIN), TOF400F3. (VIN)
- net at ACC1.GND: now also A1.J2_14 (GND), A1.J2_7 (GND), STM32_FOC1. (VIN-)
- net at ACC1.SCL: now also A1.J2_2 (D1)
- net at ACC1.SDA: now also A1.J2_3 (D2)
- net at ACC1.VCC: now also A1.J2_15 (3V3), A1.J2_6 (3V3)
- net VCC: now reaches STM32_FOC1. (VIN-)
- net VCC: now also LipoProtectionBoard1. (VOUT-), BuckConverter1. (VOUT-), BuckConverter2. (VOUT-), BuckConverter3. (VOUT-), IBT1. (VIN-), IBT4. (VIN-), STM32_FOC2. (VIN-), STM32_FOC3. (VIN-)
- net at A1.J2_8 (D5): now also STM32_FOC1. (VIN-)
- net at A1.J1_10 (GND), A1.J1_14 (GND): now also BuckConverter1. (VOUT-)
- net at A1.J1_15 (VIN): now also BuckConverter1. (VOUT-)
- net at U2.1 (VDD5V): now also STM32_FOC1. (VIN-)
- net at U2.4 (GND): now also STM32_FOC1. (VIN-)
- net at U2.6 (SDA): now also STM32_FOC1. (VIN-)
- net at U2.7 (SCL): now also STM32_FOC1. (VIN-)
- new net: A3.J2_10 (D7), IBT1. (VIN-)
- new net: A3.J2_11 (D8), IBT1. (VIN-)
- new net: A3.J2_14 (GND), A3.J2_7 (GND), ACC3.GND, STM32_FOC3. (VIN-)
- new net: A3.J2_15 (3V3), A3.J2_6 (3V3), ACC3.VCC
- new net: A3.J2_2 (D1), ACC3.SCL
- new net: A3.J2_3 (D2), ACC3.SDA
- new net: A3.J2_8 (D5), STM32_FOC3. (VIN-)
- new net: A3.J2_9 (D6), M3.2 (PWM)
- new net: A3.J1_1 (A0), M3.1 (FDBCK)
- new net: IBT1. (VIN-), M4.1 (+)
- new net: IBT1. (VIN-), M4.2 (-)
- new net: A2.J1_1 (A0), M1.1 (FDBCK)
- new net: A2.J2_9 (D6), M1.2 (PWM)
- new net: A2.J1_15 (VIN), BuckConverter2. (VOUT-), M1.3 (+)
- new net: A2.J1_10 (GND), A2.J1_14 (GND), BuckConverter2. (VOUT-), IBT4. (VIN-), M1.4 (-)
- new net: A2.J2_14 (GND), A2.J2_7 (GND), ACC2.GND, STM32_FOC2. (VIN-)
- new net: A2.J2_2 (D1), ACC2.SCL
- new net: A2.J2_3 (D2), ACC2.SDA
- new net: A2.J2_15 (3V3), A2.J2_6 (3V3), ACC2.VCC
- new net: A2.J2_10 (D7), IBT4. (VIN-)
- new net: A2.J2_11 (D8), IBT4. (VIN-)
- new net: IBT4. (VIN-), M2.1 (+)
- new net: IBT4. (VIN-), M2.2 (-)
- new net: A2.J2_8 (D5), STM32_FOC2. (VIN-)
- new net: FTDI_USB_Serial1. (VCC), U3.P$1 (5V)
- new net: FTDI_USB_Serial1. (VCC), U3.P$10 (IO1/U0T)
- new net: FTDI_USB_Serial1. (VCC), U3.P$11 (IO3/U0R)
- new net: FTDI_USB_Serial1. (VCC), U3.P$2 (GND)
- new net: PositionSensor.1 (VDD5V), STM32_FOC2. (VIN-)
- new net: PositionSensor.4 (GND), STM32_FOC2. (VIN-)
- new net: PositionSensor.6 (SDA), STM32_FOC2. (VIN-)
- new net: PositionSensor.7 (SCL), STM32_FOC2. (VIN-)
- new net: PositionSensor1.1 (VDD5V), STM32_FOC3. (VIN-)
- new net: PositionSensor1.4 (GND), STM32_FOC3. (VIN-)
- new net: PositionSensor1.6 (SDA), STM32_FOC3. (VIN-)
- new net: PositionSensor1.7 (SCL), STM32_FOC3. (VIN-)
- new net: AE1.1 (A), U1.
- new net GND: BuckConverter1. (VOUT-), BuckConverter2. (VOUT-), BuckConverter3. (VOUT-), IBT1. (VIN-), IBT4. (VIN-), LipoProtectionBoard1. (VOUT-), STM32_FOC1. (VIN-), STM32_FOC2. (VIN-), STM32_FOC3. (VIN-)
- new net MOTOR_PHASE1: STM32_FOC1. (VIN-), STM32_FOC2. (VIN-), STM32_FOC3. (VIN-)
- new net MOTOR_PHASE2: STM32_FOC1. (VIN-), STM32_FOC2. (VIN-), STM32_FOC3. (VIN-)
- new net MOTOR_PHASE3: STM32_FOC1. (VIN-), STM32_FOC2. (VIN-), STM32_FOC3. (VIN-)
- no-connect marks 0 -> 14
Other:
- note added: "5V NEEDS TO REMOVE R1"
- note added: "LIPO CIRCUIT"
- note added: "MILESTONE E SCHEMA"
- note added: "MILESTONE I SCHEMA"
- note added: "MILESTONE M SCHEMA"
- note added: "SCL"
- note added: "SDA"
- note added: "SETUP"
- moved on the sheet: A1A, A1B, ACC1, LIPO1, LipoProtectionBoard1, U2

Commit message: Edited electrical schema
Parts:
- removed A2: NodeMCU, 113990105:SEEED_113990105, symbol ESP8266:113990105
- removed IBT1, IBT4: ~, symbol MIT_Lib:IBT4
- removed PositionSensor, PositionSensor1, U2: AS5600, AS5600:AS5600, symbol AS5600:AS5600
- removed STM32_FOC2, STM32_FOC3: ~, symbol MIT_Lib:STM32_FOC
- added ATM102_ENCODER1, ATM102_ENCODER2, ATM102_ENCODER3: ~, symbol MIT_Lib:ATM102_ENCODER
- added ODRIVE_FOC2, ODRIVE_FOC3: ~, symbol MIT_Lib:ODRIVE_FOC
- added U2, U4: L298N, Package_TO_SOT_THT:TO-220-15_P2.54x2.54mm_StaggerOdd_Lead4.58mm_Vertical, symbol Driver_Motor:L298N
- added U5: ESP32-DEVKIT-V1, ESP32-DEVKIT-V1:MODULE_ESP32_DEVKIT_V1, symbol ESP32-DEVKIT:ESP32-DEVKIT-V1
- M2, M4: value Motraxx SR545SA -> YellowGearboxMotor
- ODRIVE_FOC1: renamed from STM32_FOC1; symbol MIT_Lib:STM32_FOC -> MIT_Lib:ODRIVE_FOC
Connections:
- net GND: now also ACC2.GND, M1.4 (-), ODRIVE_FOC2. (VIN-), ODRIVE_FOC3. (VIN-), U2.8 (GND), U4.8 (GND), U5.2 (GND), U5.29 (GND)
- net MOTOR_PHASE1: now also ODRIVE_FOC2. (VIN-), ODRIVE_FOC3. (VIN-)
- net MOTOR_PHASE2: now also ODRIVE_FOC2. (VIN-), ODRIVE_FOC3. (VIN-)
- net MOTOR_PHASE3: now also ODRIVE_FOC2. (VIN-), ODRIVE_FOC3. (VIN-)
- net VCC: now also ODRIVE_FOC2. (VIN-), ODRIVE_FOC3. (VIN-), U2.9 (Vss), U4.9 (Vss)
- net at A3.J2_10 (D7): now also U4.5 (IN1)
- net at A3.J2_11 (D8): now also U4.7 (IN2)
- net at A3.J2_14 (GND), A3.J2_7 (GND), ACC3.GND: now also ODRIVE_FOC3. (VIN-)
- net at A3.J1_1 (A0): no longer M3.1 (FDBCK)
- net at A1.J2_8 (D5): no longer ODRIVE_FOC1. (VIN-)
- net at M4.1 (+): now also U4.2 (OUT1)
- net at M4.2 (-): now also U4.3 (OUT2)
- net at TOF400F1. (VIN): now also TOF400F2. (VIN), TOF400F3. (VIN), U1.P$9 (.GND)
- net at M1.2 (PWM): now also U5.3 (D15)
- net at BuckConverter2. (VOUT-), M1.3 (+): now also U5.30 (VIN)
- net at ACC2.SCL: now also U5.14 (D22)
- net at ACC2.SDA: now also U5.11 (D21)
- net at ACC2.VCC: now also U5.1 (3V3)
- net at M2.1 (+): now also U2.2 (OUT1)
- net at M2.2 (-): now also U2.3 (OUT2)
- net at FTDI_USB_Serial1. (VCC): now also U3.P$2 (GND)
- new net: ATM102_ENCODER1. (X), ODRIVE_FOC1. (VIN-) (x5)
- new net: TOF400F1. (VIN), TOF400F2. (VIN), TOF400F3. (VIN), U1.P$12 (3V3.)
- new net: TOF400F1. (VIN), TOF400F2. (VIN), TOF400F3. (VIN), U1.P$5 (IO15)
- new net: TOF400F1. (VIN), TOF400F2. (VIN), TOF400F3. (VIN), U1.P$6 (IO14)
- new net: ODRIVE_FOC2. (VIN-), U5.6 (RX2)
- new net: ODRIVE_FOC2. (VIN-), U5.7 (TX2)
- new net: ATM102_ENCODER2. (X), ODRIVE_FOC2. (VIN-) (x5)
- new net: ATM102_ENCODER3. (X), ODRIVE_FOC3. (VIN-) (x5)
- now unconnected: TOF400F2. (VIN), TOF400F2. (VIN), TOF400F2. (VIN), TOF400F2. (VIN), TOF400F3. (VIN), TOF400F3. (VIN), TOF400F3. (VIN), TOF400F3. (VIN)
- no-connect marks 14 -> 15
Other:
- note removed: "5V NEEDS TO REMOVE R1"
- moved on the sheet: A3A, A3B, ACC3, AE1, BuckConverter3, M3, TOF400F1, TOF400F2, TOF400F3, U1

Commit message: Update schematic
Connections:
- net at TOF400F1. (VIN): now also TOF400F2. (VIN), TOF400F3. (VIN), U1.P$9 (.GND)
- net at ACC2.INT: now also U5.15 (D23)
- net at U2.10 (IN3): now also U5.22 (D33)
- net at U2.12 (IN4): now also U5.21 (D32)
- net at U2.13 (OUT3): now also M2.1 (+)
- net at U2.14 (OUT4): now also M2.2 (-)
- net at U2.2 (OUT1): no longer M2.1 (+)
- net at U2.3 (OUT2): no longer M2.2 (-)
- net at FTDI_USB_Serial1. (VCC): now also U3.P$2 (GND)
- new net: ATM102_ENCODER1. (X), ODRIVE_FOC1. (VIN-) (x4)
- new net: TOF400F1. (VIN), TOF400F2. (VIN), TOF400F3. (VIN), U1.P$12 (3V3.)
- new net: TOF400F1. (VIN), TOF400F2. (VIN), TOF400F3. (VIN), U1.P$5 (IO15)
- new net: TOF400F1. (VIN), TOF400F2. (VIN), TOF400F3. (VIN), U1.P$6 (IO14)
- new net: ATM102_ENCODER2. (X), ODRIVE_FOC2. (VIN-) (x4)
- new net: ATM102_ENCODER3. (X), ODRIVE_FOC3. (VIN-) (x4)
- now unconnected: TOF400F2. (VIN), TOF400F2. (VIN), TOF400F2. (VIN), TOF400F2. (VIN), TOF400F3. (VIN), TOF400F3. (VIN), TOF400F3. (VIN), TOF400F3. (VIN)
Other:
- note added: "IN3"
- note added: "IN4"
- note added: "SERVO_PWM"
- moved on the sheet: M2

Commit message: Update electrical schema
Parts:
- removed A1, A3: NodeMCU, 113990105:SEEED_113990105, symbol ESP8266:113990105
- removed ACC1, ACC3: GY-521, symbol GY-521:GY-521
- removed AE1: Antenna, symbol Device:Antenna
- removed ATM102_ENCODER1, ATM102_ENCODER3: ~, symbol MIT_Lib:ATM102_ENCODER
- removed BuckConverter1, BuckConverter3: ~, symbol MIT_Lib:Buck_Converter
- removed FTDI_USB_Serial1: ~, symbol MIT_Lib:FTDI_USB_Serial
- removed M3: DNS15, symbol Motor:Motor_Servo
- removed M4: YellowGearboxMotor, symbol Motor:Motor_DC
- removed ODRIVE_FOC1, ODRIVE_FOC3: ~, symbol MIT_Lib:ODRIVE_FOC
- removed TOF400F1, TOF400F2, TOF400F3: ~, symbol MIT_Lib:TOF400F
- removed U1, U3: ESP32-CAM, ESP32-CAM:ESP32-CAM, symbol ESP32-CAM:ESP32-CAM
- removed U4: L298N, Package_TO_SOT_THT:TO-220-15_P2.54x2.54mm_StaggerOdd_Lead4.58mm_Vertical, symbol Driver_Motor:L298N
Connections:
- new net: ATM102_ENCODER2. (X), ODRIVE_FOC2. (VIN-) (x4)
- no-connect marks 15 -> 0
Other:
- note removed: "MILESTONE E SCHEMA"
- note removed: "MILESTONE I SCHEMA"
- note removed: "MILESTONE M SCHEMA"
- note removed: "SETUP"
- moved on the sheet: ACC2, ATM102_ENCODER2, BuckConverter2, LIPO1, LipoProtectionBoard1, M1, M2, ODRIVE_FOC2, U2, U5
